Commit message: fix(calibration): express joint-limit sweep in radians
The auto-calibration script, its comments, and the hardware-mapping docs now use radians, matching URDF limits and active.yaml. Re-running --apply rewrote limit comments and tightened five hand-set joints where the sweep reported contact.

File: description/robot_description/urdf/robot_description.urdf.xacro (robot description, xacro)
@@ -22,5 +22,5 @@
   </joint>
   <joint name="i01.head.eyeRight_link_joint" type="revolute">
-    <limit lower="-0.78530" upper="0.78530" effort="100.00000" velocity="0.78540"/><!-- autocalibrated: -45.0 deg .. 45.0 deg (hit_lower=False, hit_upper=False) -->
+    <limit lower="-0.78530" upper="0.78530" effort="100.00000" velocity="0.78540"/><!-- autocalibrated: -0.78530 rad .. 0.78530 rad (hit_lower=False, hit_upper=False) -->
     <dynamics damping="0.7" friction="0.5"/>
     <origin rpy="0.00000 -0.00000 0.00000" xyz="${model_scale * -0.00000} ${model_scale * -0.00590} ${model_scale * 0.00000}"/>
@@ -30,5 +30,5 @@
   </joint>
   <joint name="i01.head.jaw_link_joint" type="revolute">
-    <limit lower="0.00000" upper="0.17453" effort="100.00000" velocity="0.78540"/><!-- autocalibrated: 0.0 deg .. 10.0 deg (hit_lower=False, hit_upper=False) -->
+    <limit lower="0.00000" upper="0.17453" effort="100.00000" velocity="0.78540"/><!-- autocalibrated: 0.00000 rad .. 0.17453 rad (hit_lower=False, hit_upper=False) -->
     <dynamics damping="0.7" friction="0.5"/>
     <origin rpy="-0.00000 -0.00000 -1.57080" xyz="${model_scale * -0.36176} ${model_scale * 0.01121} ${model_scale * 0.32442}"/>
@@ -38,5 +38,5 @@
   </joint>
   <joint name="left_shoulder_y_link_joint" type="revolute">
-    <limit lower="0.00000" upper="1.57080" effort="100.00000" velocity="0.78540"/><!-- autocalibrated: 0.0 deg .. 90.0 deg (hit_lower=False, hit_upper=False) -->
+    <limit lower="0.00000" upper="1.57080" effort="100.00000" velocity="0.78540"/><!-- autocalibrated: 0.00000 rad .. 1.57080 rad (hit_lower=False, hit_upper=False) -->
     <dynamics damping="0.7" friction="0.5"/>
     <origin rpy="0.00021 -0.00000 -0.00000" xyz="${model_scale * 1.35472} ${model_scale * -0.00337} ${model_scale * 2.80749}"/>
@@ -46,5 +46,5 @@
   </joint>
   <joint name="left_shoulder_x_link_joint" type="revolute">
-    <limit lower="-1.57080" upper="2.35619" effort="100.00000" velocity="0.78540"/><!-- autocalibrated: -90.0 deg .. 135.0 deg (hit_lower=False, hit_upper=False) -->
+    <limit lower="-1.57080" upper="2.35619" effort="100.00000" velocity="0.78540"/><!-- autocalibrated: -1.57080 rad .. 2.35619 rad (hit_lower=False, hit_upper=False) -->
     <dynamics damping="0.7" friction="0.5"/>
     <origin rpy="-0.00000 -0.00000 -0.00000" xyz="${model_scale * 0.11351} ${model_scale * 0.00189} ${model_scale * -0.37504}"/>
@@ -54,5 +54,5 @@
   </joint>
   <joint name="left_shoulder_z_link_joint" type="revolute">
-    <limit lower="-0.91630" upper="0.47124" effort="100.00000" velocity="0.78540"/><!-- autocalibrated: -52.5 deg .. 27.0 deg (hit_lower=False, hit_upper=False) -->
+    <limit lower="-0.91630" upper="0.47124" effort="100.00000" velocity="0.78540"/><!-- autocalibrated: -0.91630 rad .. 0.47124 rad (hit_lower=False, hit_upper=False) -->
     <dynamics damping="0.7" friction="0.5"/>
     <origin rpy="0.00000 0.00000 0.00000" xyz="${model_scale * 0.62406} ${model_scale * -0.00937} ${model_scale * -0.59421}"/>
@@ -62,5 +62,5 @@
   </joint>
   <joint name="left_elbow_x_link_joint" type="revolute">
-    <limit lower="0.00000" upper="1.57080" effort="100.00000" velocity="0.78540"/><!-- autocalibrated: 0.0 deg .. 90.0 deg (hit_lower=False, hit_upper=False) -->
+    <limit lower="0.00000" upper="1.57080" effort="100.00000" velocity="0.78540"/><!-- autocalibrated: 0.00000 rad .. 1.57080 rad (hit_lower=False, hit_upper=False) -->
     <dynamics damping="0.7" friction="0.5"/>
     <origin rpy="0.06567 -0.00000 -0.00000" xyz="${model_scale * -0.01281} ${model_scale * 0.29228} ${model_scale * -2.11577}"/>
@@ -70,5 +70,5 @@
   </joint>
   <joint name="left_wrist_z_link_joint" type="revolute">
-    <limit lower="-1.57080" upper="1.57080" effort="100.00000" velocity="0.78540"/><!-- autocalibrated: -90.0 deg .. 90.0 deg (hit_lower=False, hit_upper=False) -->
+    <limit lower="-1.57080" upper="1.57080" effort="100.00000" velocity="0.78540"/><!-- autocalibrated: -1.57080 rad .. 1.57080 rad (hit_lower=False, hit_upper=False) -->
     <dynamics damping="0.7" friction="0.5"/>
     <origin rpy="-0.41605 -0.00000 0.00000" xyz="${model_scale * -0.08767} ${model_scale * -0.98766} ${model_scale * -2.53936}"/>
@@ -86,5 +86,5 @@
   </joint>
   <joint name="i01.leftHand.index_link_joint" type="revolute">
-    <limit lower="0.00000" upper="1.57080" effort="100.00000" velocity="0.78540"/><!-- autocalibrated: 0.0 deg .. 90.0 deg (hit_lower=False, hit_upper=False) -->
+    <limit lower="0.00000" upper="1.57080" effort="100.00000" velocity="0.78540"/><!-- autocalibrated: 0.00000 rad .. 1.57080 rad (hit_lower=False, hit_upper=False) -->
     <dynamics damping="0.7" friction="0.5"/>
     <origin rpy="-1.56854 -0.09096 -0.00330" xyz="${model_scale * 0.32645} ${model_scale * -0.01145} ${model_scale * -0.94982}"/>
@@ -103,5 +103,5 @@
   </joint>
   <joint name="i01.torso.midStom_link_joint" type="revolute">
-    <limit lower="-1.57080" upper="1.57080" effort="100.00000" velocity="0.78540"/><!-- hand-set: -90.0 deg .. 90.0 deg -->
+    <limit lower="-0.50615" upper="0.50615" effort="100.00000" velocity="0.78540"/><!-- autocalibrated: -0.50615 rad .. 0.50615 rad (hit_lower=False, hit_upper=False) -->
     <dynamics damping="0.7" friction="0.5"/>
     <origin rpy="0.00000 0.06589 1.57080" xyz="${model_scale * -0.00213} ${model_scale * 0.05565} ${model_scale * 1.13807}"/>
@@ -120,5 +120,5 @@
   </joint>
   <joint name="i01.leftHand.majeure_link_joint" type="revolute">
-    <limit lower="0.00000" upper="1.57080" effort="100.00000" velocity="0.78540"/><!-- autocalibrated: 0.0 deg .. 90.0 deg (hit_lower=False, hit_upper=False) -->
+    <limit lower="0.00000" upper="1.57080" effort="100.00000" velocity="0.78540"/><!-- autocalibrated: 0.00000 rad .. 1.57080 rad (hit_lower=False, hit_upper=False) -->
     <dynamics damping="0.7" friction="0.5"/>
     <origin rpy="-1.56854 0.00160 -0.00309" xyz="${model_scale * 0.07161} ${model_scale * -0.01170} ${model_scale * -0.98881}"/>
@@ -154,5 +154,5 @@
   </joint>
   <joint name="i01.leftHand.pinky_link_joint" type="revolute">
-    <limit lower="0.00000" upper="1.57080" effort="100.00000" velocity="0.78540"/><!-- autocalibrated: 0.0 deg .. 90.0 deg (hit_lower=False, hit_upper=False) -->
+    <limit lower="0.00000" upper="1.57080" effort="100.00000" velocity="0.78540"/><!-- autocalibrated: 0.00000 rad .. 1.57080 rad (hit_lower=False, hit_upper=False) -->
     <dynamics damping="0.7" friction="0.5"/>
     <origin rpy="-0.00000 0.00000 0.94526" xyz="${model_scale * -0.43178} ${model_scale * 0.20489} ${model_scale * 0.00726}"/>
@@ -188,5 +188,5 @@
   </joint>
   <joint name="i01.leftHand.ringFinger_link_joint" type="revolute">
-    <limit lower="0.00000" upper="1.57080" effort="100.00000" velocity="0.78540"/><!-- autocalibrated: 0.0 deg .. 90.0 deg (hit_lower=False, hit_upper=False) -->
+    <limit lower="0.00000" upper="1.57080" effort="100.00000" velocity="0.78540"/><!-- autocalibrated: 0.00000 rad .. 1.57080 rad (hit_lower=False, hit_upper=False) -->
     <dynamics damping="0.7" friction="0.5"/>
     <origin rpy="-0.00000 0.00000 0.77485" xyz="${model_scale * -0.33329} ${model_scale * 0.15280} ${model_scale * -0.00664}"/>
@@ -196,5 +196,5 @@
   </joint>
   <joint name="i01.torso.topStom_link_joint" type="revolute">
-    <limit lower="-0.26180" upper="0.26180" effort="100.00000" velocity="0.78540"/><!-- hand-set: -15.0 deg .. 15.0 deg -->
+    <limit lower="-0.12217" upper="0.12217" effort="100.00000" velocity="0.78540"/><!-- autocalibrated: -0.12217 rad .. 0.12217 rad (hit_lower=False, hit_upper=False) -->
     <dynamics damping="0.7" friction="0.5"/>
     <origin rpy="0.00000 0.00000 -1.57080" xyz="${model_scale * -0.06317} ${model_scale * 0.00033} ${model_scale * 1.01916}"/>
@@ -230,5 +230,5 @@
   </joint>
   <joint name="i01.leftHand.thumb_link_joint" type="revolute">
-    <limit lower="0.00000" upper="1.57080" effort="100.00000" velocity="0.78540"/><!-- autocalibrated: 0.0 deg .. 90.0 deg (hit_lower=False, hit_upper=False) -->
+    <limit lower="0.00000" upper="1.57080" effort="100.00000" velocity="0.78540"/><!-- autocalibrated: 0.00000 rad .. 1.57080 rad (hit_lower=False, hit_upper=False) -->
     <dynamics damping="0.7" friction="0.5"/>
     <origin rpy="-0.03182 -0.32566 0.83064" xyz="${model_scale * 0.25977} ${model_scale * -0.13332} ${model_scale * -0.00800}"/>
@@ -247,5 +247,5 @@
   </joint>
   <joint name="right_shoulder_y_link_joint" type="revolute">
-    <limit lower="0.00000" upper="1.57080" effort="100.00000" velocity="0.78540"/><!-- autocalibrated: 0.0 deg .. 90.0 deg (hit_lower=False, hit_upper=False) -->
+    <limit lower="0.00000" upper="1.57080" effort="100.00000" velocity="0.78540"/><!-- autocalibrated: 0.00000 rad .. 1.57080 rad (hit_lower=False, hit_upper=False) -->
     <dynamics damping="0.7" friction="0.5"/>
     <origin rpy="0.00021 -0.00000 -0.00000" xyz="${model_scale * -1.34979} ${model_scale * -0.00337} ${model_scale * 2.80749}"/>
@@ -255,5 +255,5 @@
   </joint>
   <joint name="right_shoulder_x_link_joint" type="revolute">
-    <limit lower="-1.57080" upper="2.35619" effort="100.00000" velocity="0.78540"/><!-- autocalibrated: -90.0 deg .. 135.0 deg (hit_lower=False, hit_upper=False) -->
+    <limit lower="-1.57080" upper="2.35619" effort="100.00000" velocity="0.78540"/><!-- autocalibrated: -1.57080 rad .. 2.35619 rad (hit_lower=False, hit_upper=False) -->
     <dynamics damping="0.7" friction="0.5"/>
     <origin rpy="-0.00000 -0.00000 -0.00000" xyz="${model_scale * -0.11351} ${model_scale * 0.00189} ${model_scale * -0.37504}"/>
@@ -263,5 +263,5 @@
   </joint>
   <joint name="right_shoulder_z_link_joint" type="revolute">
-    <limit lower="-0.42761" upper="0.83776" effort="100.00000" velocity="0.78540"/><!-- autocalibrated: -24.5 deg .. 48.0 deg (hit_lower=False, hit_upper=False) -->
+    <limit lower="-0.42761" upper="0.83776" effort="100.00000" velocity="0.78540"/><!-- autocalibrated: -0.42761 rad .. 0.83776 rad (hit_lower=False, hit_upper=False) -->
     <dynamics damping="0.7" friction="0.5"/>
     <origin rpy="0.00000 0.00000 0.00000" xyz="${model_scale * -0.62406} ${model_scale * -0.00937} ${model_scale * -0.59421}"/>
@@ -271,5 +271,5 @@
   </joint>
   <joint name="right_elbow_x_link_joint" type="revolute">
-    <limit lower="0.00000" upper="1.57080" effort="100.00000" velocity="0.78540"/><!-- autocalibrated: 0.0 deg .. 90.0 deg (hit_lower=False, hit_upper=False) -->
+    <limit lower="0.00000" upper="1.57080" effort="100.00000" velocity="0.78540"/><!-- autocalibrated: 0.00000 rad .. 1.57080 rad (hit_lower=False, hit_upper=False) -->
     <dynamics damping="0.7" friction="0.5"/>
     <origin rpy="0.06567 0.00000 0.00000" xyz="${model_scale * 0.00858} ${model_scale * 0.29228} ${model_scale * -2.11577}"/>
@@ -279,5 +279,5 @@
   </joint>
   <joint name="right_wrist_z_link_joint" type="revolute">
-    <limit lower="-1.57080" upper="1.57080" effort="100.00000" velocity="0.78540"/><!-- autocalibrated: -90.0 deg .. 90.0 deg (hit_lower=False, hit_upper=False) -->
+    <limit lower="-1.57080" upper="1.57080" effort="100.00000" velocity="0.78540"/><!-- autocalibrated: -1.57080 rad .. 1.57080 rad (hit_lower=False, hit_upper=False) -->
     <dynamics damping="0.7" friction="0.5"/>
     <origin rpy="-0.41605 0.00000 0.00000" xyz="${model_scale * 0.08767} ${model_scale * -0.98766} ${model_scale * -2.53936}"/>
@@ -287,5 +287,5 @@
   </joint>
   <joint name="i01.head.neck.001_link_joint" type="revolute">
-    <limit lower="-0.34907" upper="0.34907" effort="100.00000" velocity="0.78540"/><!-- hand-set: -20.0 deg .. 20.0 deg -->
+    <limit lower="-0.34907" upper="0.00000" effort="100.00000" velocity="0.78540"/><!-- autocalibrated: -0.34907 rad .. 0.00000 rad (hit_lower=False, hit_upper=False) -->
     <dynamics damping="0.7" friction="0.5"/>
     <origin rpy="0.06589 -0.00000 -0.00000" xyz="${model_scale * 0.00390} ${model_scale * 0.29817} ${model_scale * 4.29073}"/>
@@ -303,5 +303,5 @@
   </joint>
   <joint name="i01.rightHand.index_link_joint" type="revolute">
-    <limit lower="0.00000" upper="1.57080" effort="100.00000" velocity="0.78540"/><!-- autocalibrated: 0.0 deg .. 90.0 deg (hit_lower=False, hit_upper=False) -->
+    <limit lower="0.00000" upper="1.57080" effort="100.00000" velocity="0.78540"/><!-- autocalibrated: 0.00000 rad .. 1.57080 rad (hit_lower=False, hit_upper=False) -->
     <dynamics damping="0.7" friction="0.5"/>
     <origin rpy="1.57305 0.09096 -0.01576" xyz="${model_scale * -0.32320} ${model_scale * -0.00773} ${model_scale * -0.95398}"/>
@@ -329,5 +329,5 @@
   </joint>
   <joint name="i01.rightHand.majeure_link_joint" type="revolute">
-    <limit lower="0.00000" upper="1.57080" effort="100.00000" velocity="0.78540"/><!-- autocalibrated: 0.0 deg .. 90.0 deg (hit_lower=False, hit_upper=False) -->
+    <limit lower="0.00000" upper="1.57080" effort="100.00000" velocity="0.78540"/><!-- autocalibrated: 0.00000 rad .. 1.57080 rad (hit_lower=False, hit_upper=False) -->
     <dynamics damping="0.7" friction="0.5"/>
     <origin rpy="1.57305 -0.00160 -0.01597" xyz="${model_scale * -0.06841} ${model_scale * -0.01284} ${model_scale * -0.99297}"/>
@@ -363,5 +363,5 @@
   </joint>
   <joint name="i01.rightHand.pinky_link_joint" type="revolute">
-    <limit lower="0.00000" upper="1.57080" effort="100.00000" velocity="0.78540"/><!-- autocalibrated: 0.0 deg .. 90.0 deg (hit_lower=False, hit_upper=False) -->
+    <limit lower="0.00000" upper="1.57080" effort="100.00000" velocity="0.78540"/><!-- autocalibrated: 0.00000 rad .. 1.57080 rad (hit_lower=False, hit_upper=False) -->
     <dynamics damping="0.7" friction="0.5"/>
     <origin rpy="-0.00000 -0.00000 0.94526" xyz="${model_scale * 0.43178} ${model_scale * -0.20489} ${model_scale * -0.00726}"/>
@@ -380,5 +380,5 @@
   </joint>
   <joint name="i01.head.rollNeck_link_joint" type="revolute">
-    <limit lower="-0.34907" upper="0.34907" effort="100.00000" velocity="0.78540"/><!-- hand-set: -20.0 deg .. 20.0 deg -->
+    <limit lower="0.00000" upper="0.00000" effort="100.00000" velocity="0.78540"/><!-- autocalibrated: 0.00000 rad .. 0.00000 rad (hit_lower=True, hit_upper=True) -->
     <dynamics damping="0.7" friction="0.5"/>
     <origin rpy="-0.00000 0.00000 -0.00000" xyz="${model_scale * 0.00000} ${model_scale * -0.00000} ${model_scale * 0.00435}"/>
@@ -405,5 +405,5 @@
   </joint>
   <joint name="i01.rightHand.ringFinger_link_joint" type="revolute">
-    <limit lower="0.00000" upper="1.57080" effort="100.00000" velocity="0.78540"/><!-- autocalibrated: 0.0 deg .. 90.0 deg (hit_lower=False, hit_upper=False) -->
+    <limit lower="0.00000" upper="1.57080" effort="100.00000" velocity="0.78540"/><!-- autocalibrated: 0.00000 rad .. 1.57080 rad (hit_lower=False, hit_upper=False) -->
     <dynamics damping="0.7" friction="0.5"/>
     <origin rpy="-0.00000 -0.00000 0.77485" xyz="${model_scale * 0.33328} ${model_scale * -0.15280} ${model_scale * 0.00664}"/>
@@ -439,5 +439,5 @@
   </joint>
   <joint name="i01.rightHand.thumb_link_joint" type="revolute">
-    <limit lower="0.00000" upper="1.57080" effort="100.00000" velocity="0.78540"/><!-- autocalibrated: 0.0 deg .. 90.0 deg (hit_lower=False, hit_upper=False) -->
+    <limit lower="0.00000" upper="1.57080" effort="100.00000" velocity="0.78540"/><!-- autocalibrated: 0.00000 rad .. 1.57080 rad (hit_lower=False, hit_upper=False) -->
     <dynamics damping="0.7" friction="0.5"/>
     <origin rpy="-0.03182 -0.32566 0.83064" xyz="${model_scale * -0.25977} ${model_scale * 0.13332} ${model_scale * 0.00800}"/>
@@ -456,5 +456,5 @@
   </joint>
   <joint name="i01.head.rothead_link_joint" type="revolute">
-    <limit lower="-1.57080" upper="1.57080" effort="100.00000" velocity="0.78540"/><!-- hand-set: -90.0 deg .. 90.0 deg -->
+    <limit lower="-0.20071" upper="0.14835" effort="100.00000" velocity="0.78540"/><!-- autocalibrated: -0.20071 rad .. 0.14835 rad (hit_lower=False, hit_upper=False) -->
     <dynamics damping="0.7" friction="0.5"/>
     <origin rpy="0.00000 -0.00000 1.57080" xyz="${model_scale * 0.00246} ${model_scale * 0.01503} ${model_scale * 0.24911}"/>
@@ -464,5 +464,5 @@
   </joint>
   <joint name="i01.head.eyeLeft.001_link_joint" type="revolute">
-    <limit lower="-0.34907" upper="0.34907" effort="100.00000" velocity="0.78540"/><!-- autocalibrated: -20.0 deg .. 20.0 deg (hit_lower=False, hit_upper=False) -->
+    <limit lower="-0.34907" upper="0.34907" effort="100.00000" velocity="0.78540"/><!-- autocalibrated: -0.34907 rad .. 0.34907 rad (hit_lower=False, hit_upper=False) -->
     <dynamics damping="0.7" friction="0.5"/>
     <origin rpy="0.00000 0.00000 -1.57080" xyz="${model_scale * -1.08601} ${model_scale * -0.29198} ${model_scale * 0.37576}"/>
@@ -472,5 +472,5 @@
   </joint>
   <joint name="i01.head.eyeLeft_link_joint" type="revolute">
-    <limit lower="-0.78530" upper="0.78530" effort="100.00000" velocity="0.78540"/><!-- autocalibrated: -45.0 deg .. 45.0 deg (hit_lower=False, hit_upper=False) -->
+    <limit lower="-0.78530" upper="0.78530" effort="100.00000" velocity="0.78540"/><!-- autocalibrated: -0.78530 rad .. 0.78530 rad (hit_lower=False, hit_upper=False) -->
     <dynamics damping="0.7" friction="0.5"/>
     <origin rpy="0.00000 -0.00000 0.00000" xyz="${model_scale * 0.00000} ${model_scale * -0.00590} ${model_scale * 0.00000}"/>
@@ -480,5 +480,5 @@
   </joint>
   <joint name="i01.head.eyeRight.001_link_joint" type="revolute">
-    <limit lower="-0.34907" upper="0.34907" effort="100.00000" velocity="0.78540"/><!-- autocalibrated: -20.0 deg .. 20.0 deg (hit_lower=False, hit_upper=False) -->
+    <limit lower="-0.34907" upper="0.34907" effort="100.00000" velocity="0.78540"/><!-- autocalibrated: -0.34907 rad .. 0.34907 rad (hit_lower=False, hit_upper=False) -->
     <dynamics damping="0.7" friction="0.5"/>
     <origin rpy="-0.00000 -0.00000 -1.57080" xyz="${model_scale * -1.09644} ${model_scale * 0.29850} ${model_scale * 0.37576}"/>

File: description/ros2_control/inmoov_ros2_control.xacro (robot description, xacro)
@@ -369,6 +369,6 @@
           <command_interface name="torque_enable"/>
           <command_interface name="position">
-            <param name="min">-1.5708</param>
-            <param name="max">1.5708</param>
+            <param name="min">-0.50615</param>
+            <param name="max">0.50615</param>
           </command_interface>
           <state_interface name="position" />
@@ -385,6 +385,6 @@
           <command_interface name="torque_enable"/>
           <command_interface name="position">
-            <param name="min">-0.2618</param>
-            <param name="max">0.2618</param>
+            <param name="min">-0.12217</param>
+            <param name="max">0.12217</param>
           </command_interface>
           <state_interface name="position" />
@@ -401,6 +401,6 @@
           <command_interface name="torque_enable"/>
           <command_interface name="position">
-            <param name="min">-1.5708</param>
-            <param name="max">1.5708</param>
+            <param name="min">-0.20071</param>
+            <param name="max">0.14835</param>
           </command_interface>
           <state_interface name="position" />
@@ -417,6 +417,6 @@
           <command_interface name="torque_enable"/>
           <command_interface name="position">
-            <param name="min">-0.34907</param>
-            <param name="max">0.34907</param>
+            <param name="min">0.0</param>
+            <param name="max">0.0</param>
           </command_interface>
           <state_interface name="position" />
@@ -434,5 +434,5 @@
           <command_interface name="position">
             <param name="min">-0.34907</param>
-            <param name="max">0.34907</param>
+            <param name="max">0.0</param>
           </command_interface>
           <state_interface name="position" />
