Commit message: fix(gazebo): drop the stand anchoring the world joint replaced

File: description/gazebo/inmoov_gazebo_physics.xacro (robot description, xacro)
@@ -26,7 +26,4 @@
     <origin xyz="0 0 0.02" rpy="0 0 0"/>
   </joint>
-  <gazebo reference="stand_link">
-    <static>true</static>
-  </gazebo>
   <!-- Body links: full-mesh collisions with self-collision disabled. Adjacent
        shoulder/elbow meshes overlap at neutral pose; enabling self-collide

File: description/robot_description/urdf/robot_description.urdf.xacro (robot description, xacro)
@@ -1,5 +1,5 @@
 <?xml version="1.0"?>
 <robot xmlns:xacro="http://www.ros.org/wiki/xacro" name="inmoov" version="1.0">
-  <!-- mesh_dir and use_gazebo_sim set by parent (inmoov.urdf.xacro) -->
+  <!-- mesh_dir set by parent (inmoov.urdf.xacro) -->
   <material name="white">
     <color rgba="1.0 1.0 1.0 1.0"/>
@@ -506,12 +506,6 @@
     </collision>
     <inertial>
-      <xacro:if value="${use_gazebo_sim}">
-        <mass value="10000"/>
-        <inertia ixx="100" ixy="0" ixz="0" iyy="100" iyz="0" izz="100"/>
-      </xacro:if>
-      <xacro:unless value="${use_gazebo_sim}">
-        <mass value="0.001"/>
-        <inertia ixx="1e-6" ixy="0" ixz="0" iyy="1e-6" iyz="0" izz="1e-6"/>
-      </xacro:unless>
+      <mass value="0.001"/>
+      <inertia ixx="1e-6" ixy="0" ixz="0" iyy="1e-6" iyz="0" izz="1e-6"/>
     </inertial>
   </link>
@@ -528,12 +522,6 @@
     </collision>
     <inertial>
-      <xacro:if value="${use_gazebo_sim}">
-        <mass value="10000"/>
-        <inertia ixx="100" ixy="0" ixz="0" iyy="100" iyz="0" izz="100"/>
-      </xacro:if>
-      <xacro:unless value="${use_gazebo_sim}">
-        <mass value="0.001"/>
-        <inertia ixx="1e-6" ixy="0" ixz="0" iyy="1e-6" iyz="0" izz="1e-6"/>
-      </xacro:unless>
+      <mass value="0.001"/>
+      <inertia ixx="1e-6" ixy="0" ixz="0" iyy="1e-6" iyz="0" izz="1e-6"/>
     </inertial>
   </link>

File: description/urdf/inmoov.urdf.xacro (robot description, xacro)
@@ -10,8 +10,7 @@
   <xacro:arg name="ros2_control_file" default="inmoov_ros2_control.xacro"/>
   <xacro:property name="mesh_dir" value="file://$(arg base_path)/robot_description/meshes/dae"/>
-  <xacro:property name="use_gazebo_sim" value="$(arg use_gazebo_sim)"/>
   <!-- model_scale lives in properties.xacro; not a launch argument. -->
   <xacro:include filename="../robot_description/urdf/properties.xacro"/>
-  <!-- Import inmoov physical description (urdf) macro (uses use_gazebo_sim for heavy stand in sim) -->
+  <!-- Import inmoov physical description (urdf) macro -->
   <xacro:include filename="../robot_description/urdf/robot_description.urdf.xacro"/>
   <!-- Import inmoov ros2_control description for real/mock hardware only.
@@ -25,5 +24,5 @@
   <!-- Gazebo-only bits, gated on use_gazebo_sim:=true:
          - gazebo/inmoov_gazebo_physics.xacro    physics + surface tuning
-                                                 (static stand, friction, self_collide, kp/kd)
+                                                 (world anchor, friction, self_collide, kp/kd)
          - gazebo/gazebo.xacro                   generated gz_ros2_control plugin +
                                                  camera sensors so the same controllers
